Commit message: smoothed out janky simulator wheel phyiscs

File: src/AutoCarROS2/autocar_description/urdf/autocar.xacro (robot description, xacro)
@@ -1,4 +1,5 @@
 <?xml version="1.0"?>
 <robot name="autocar" xmlns:xacro="http://www.ros.org/wiki/xacro">
+  <xacro:include filename="$(find autocar_description)/urdf/_d415.urdf.xacro" />
   <!-- RVIZ MATERIAL COLOUR -->
   <material name="silver">
@@ -46,4 +47,7 @@
     </inertial>
   </link>
+  <xacro:sensor_d415 parent="realsense_link">
+    <origin xyz="0 0 0" rpy="1.5708 -1.5708 0"/>
+  </xacro:sensor_d415>
   <link name="imu_link">
     <visual>
