Commit message: minor changes

File: src/AutoCarROS2/autocar_description/urdf/autocar.urdf (robot description, URDF)
Before this commit: robot autocar, 20 links, 19 joints
Links:
- link chassis_link: geometry collision mesh filename=package://autocar_description/meshes/zamboni_no_cond.stl scale=0.001 0.001 0.001; visual mesh filename=package://autocar_description/meshes/zamboni_no_cond.stl scale=0.001 0.001 0.001

File: src/AutoCarROS2/autocar_description/urdf/autocar.xacro (robot description, xacro)
@@ -70,14 +70,14 @@
     </inertial>
     <visual>
+      <origin rpy="0 0 0" xyz="0 0 -0.4" />
+      <geometry>
+        <mesh filename="package://autocar_description/meshes/zamboni_no_cond.stl" scale="0.001 0.001 0.001" />
+      </geometry>
+      <material name="silver" />
+    </visual>
+    <collision>
       <origin rpy="0 0 0" xyz="0 0 0" />
       <geometry>
-        <mesh filename="package://autocar_description/meshes/zamboni2.stl" scale="0.001 0.001 0.001" />
-      </geometry>
-      <material name="silver" />
-    </visual>
-    <collision>
-      <origin rpy="0 0 0" xyz="0 0 0" />
-      <geometry>
-        <mesh filename="package://autocar_description/meshes/zamboni2.stl" scale="0.001 0.001 0.001" />
+        <mesh filename="package://autocar_description/meshes/zamboni_no_cond.stl" scale="0.001 0.001 0.001" />
       </geometry>
     </collision>
